Commit message: Fix frictions for wheels to allow robot to move properly

File: my_rb1_description/urdf/my_rb1_robot.urdf (robot description, URDF)
Before this commit: robot RB1, 7 links, 6 joints
Links:
- added link dummy_link
Joints:
- added joint base_joint: type fixed, parent dummy_link, child base_link, origin xyz=0 0 0.15 rpy=0 0 0
- joint joint_base_back_caster: limit effort=10000 velocity=1000 -> (none)
- joint joint_base_front_caster: limit effort=10000 velocity=1000 -> (none)
- joint joint_base_front_laser: limit effort=10000 velocity=1000 -> (none)
- joint joint_base_left_wheel: limit effort=10000 velocity=1000 -> (none)
- joint joint_base_right_wheel: limit effort=10000 velocity=1000 -> (none)
